File: THT/Hardware/SmartRV-AIO-THT.kicad_sch (KiCad schematic)
At the start: 56 parts, among them J1 Programming Header, J10 Temp 4, J11 Water Level Sensor, J12 Water Level Sensor, J13 Water Level Sensor, J14 Screw_Terminal_01x02, J15 Screw_Terminal_01x02, J16 Screw_Terminal_01x02, J17 Screw_Terminal_01x02, J18 Screw_Terminal_01x02, J19 Screw_Terminal_01x03, J2 Button1, J20 Screw_Terminal_01x03, J3 Button2, J4 Button3, J5 Button4, J6 Screw_Terminal_01x02, J7 Temp 1, J8 Temp 2, J9 Temp 3, K1 Relay, K2 Relay, K3 Relay, K4 Relay, K5 Relay, K6 Relay, K7 Relay, Q1 MMBT2222A, Q2 MMBT2222A, U1 ESP32-WROOM-32D, U2 AMS1117-3.3, U3 ULN2003A

Commit message: updated schematic and images
Parts:
- removed C1: 100nf, Capacitor_SMD:C_0805_2012Metric, symbol Device:C_Small
- removed C10: 22uF, Capacitor_SMD:C_0805_2012Metric, symbol Device:C_Small
- removed C11, C4, C7, C8, C9: TBC, Capacitor_SMD:C_0805_2012Metric, symbol Device:C_Small
- removed C2: 10uF, Capacitor_SMD:C_0805_2012Metric, symbol Device:C_Small
- removed C3: 0.1uF, Capacitor_SMD:C_0805_2012Metric, symbol Device:C_Small
- removed D1: SS14, SamacSys_Parts:DIOM5126X250N, symbol SamacSys_Parts:SS14
- removed J10: Temp 4, Connector_JST:JST_XH_B3B-XH-A_1x03_P2.50mm_Vertical, symbol Connector_Generic:Conn_01x03
- removed J18: Screw_Terminal_01x02, TerminalBlock_Phoenix:TerminalBlock_Phoenix_MKDS-1,5-2_1x02_P5.00mm_Horizontal, symbol Connector:Screw_Terminal_01x02
- removed Q1, Q2: MMBT2222A, SamacSys_Parts:SOT95P240X120-3N, symbol SamacSys_Parts:MMBT2222A
- removed R1, R2, R3: 10k, Resistor_SMD:R_0805_2012Metric, symbol Device:R
- removed R8: 470, Resistor_SMD:R_0805_2012Metric, symbol Device:R
- removed U1: ESP32-WROOM-32D, RF_Module:ESP32-WROOM-32, symbol RF_Module:ESP32-WROOM-32D
- removed U2: AMS1117-3.3, Package_TO_SOT_SMD:SOT-223-3_TabPin2, symbol Regulator_Linear:AMS1117-3.3
- removed U3: ULN2003A, uln:SOIC127P600X175-16N, symbol Transistor_Array:ULN2003A
- added D1: 1N4148, Diode_THT:D_DO-35_SOD27_P7.62mm_Horizontal, symbol Diode:1N4148
- added J11, J19, J24: Screw_Terminal_01x03, TerminalBlock_Phoenix:TerminalBlock_Phoenix_MKDS-1,5-3_1x03_P5.00mm_Horizontal, symbol Connector:Screw_Terminal_01x03
- added J22, J23: Screw_Terminal_01x02, TerminalBlock_Phoenix:TerminalBlock_Phoenix_MKDS-1,5-2_1x02_P5.00mm_Horizontal, symbol Connector:Screw_Terminal_01x02
- added J5: RJ45, Connector_RJ:RJ45_Amphenol_54602-x08_Horizontal, symbol Connector:RJ45
- added Q1, Q2: 2N3904, Package_TO_SOT_THT:TO-92_Inline, symbol Transistor_BJT:2N3904
- added Q3, Q4: IRF540N, Package_TO_SOT_THT:TO-220-3_Vertical, symbol Transistor_FET:IRF540N
- added R10, R11: 470, Resistor_THT:R_Axial_DIN0207_L6.3mm_D2.5mm_P7.62mm_Horizontal, symbol Device:R
- added R12, R13, R5, R9: 10k, Resistor_THT:R_Axial_DIN0207_L6.3mm_D2.5mm_P7.62mm_Horizontal, symbol Device:R
- added U1: mini_esp32, ESP32_mini:ESP32_mini, symbol ESP32_mini:mini_esp32
- added U2: MCP23008-xP, Package_DIP:DIP-18_W7.62mm, symbol Interface_Expansion:MCP23008-xP
- added U3: ULN2003, Package_DIP:DIP-16_W7.62mm_LongPads, symbol Transistor_Array:ULN2003
- C1: renamed from C5; footprint Capacitor_SMD:C_0805_2012Metric -> Capacitor_THT:C_Disc_D5.1mm_W3.2mm_P5.00mm
- C2: renamed from C6; footprint Capacitor_SMD:C_0805_2012Metric -> Capacitor_THT:C_Radial_D5.0mm_H5.0mm_P2.00mm
- R1: renamed from R5; footprint Resistor_SMD:R_0805_2012Metric -> Resistor_THT:R_Axial_DIN0207_L6.3mm_D2.5mm_P7.62mm_Horizontal
- R2: renamed from R6; footprint Resistor_SMD:R_0805_2012Metric -> Resistor_THT:R_Axial_DIN0207_L6.3mm_D2.5mm_P7.62mm_Horizontal
- R3: renamed from R7; footprint Resistor_SMD:R_0805_2012Metric -> Resistor_THT:R_Axial_DIN0207_L6.3mm_D2.5mm_P7.62mm_Horizontal
- R4: footprint Resistor_SMD:R_0805_2012Metric -> Resistor_THT:R_Axial_DIN0207_L6.3mm_D2.5mm_P7.62mm_Horizontal
- R6: renamed from R9; footprint Resistor_SMD:R_0805_2012Metric -> Resistor_THT:R_Axial_DIN0207_L6.3mm_D2.5mm_P7.62mm_Horizontal
- R7: renamed from R10; footprint Resistor_SMD:R_0805_2012Metric -> Resistor_THT:R_Axial_DIN0207_L6.3mm_D2.5mm_P7.62mm_Horizontal
- R8: renamed from R11; footprint Resistor_SMD:R_0805_2012Metric -> Resistor_THT:R_Axial_DIN0207_L6.3mm_D2.5mm_P7.62mm_Horizontal
- renumbered J9 to J10, J11 to J12, J12 to J13, J13 to J14, J14 to J15, J15 to J16, J16 to J17, J17 to J18, J19 to J20, J20 to J21, J5 to J6, J6 to J7, J7 to J8, J8 to J9
Connections:
- net 12v: now also J22.1 (Pin_1), J23.2 (Pin_2)
- net 3v3: now also J10.1 (Pin_1), J8.1 (Pin_1), J9.1 (Pin_1), R1.1, R2.1, R3.1, J11.1 (Pin_1), J19.1 (Pin_1), R5.1, R9.1, U1.16 (3V3), U2.18 (VDD)
- net 5v: now also J5.1, J5.2, U1.35 (VCC_(USB)), U3.9 (COM)
- net Button1: now also U1.24 (IO_27)
- net Button2: now also U1.6 (IO_26/D0)
- net Button3: now also U1.26 (IO_25)
- net Button4: now also U1.12 (IO_23/D7)
- net ESP_RX: now also U1.23 (RXD)
- net ESP_TX: now also U1.21 (TXD)
- net GND: now also J11.3 (Pin_3), J19.3 (Pin_3), J5.3, J5.4, Q1.1 (E), Q2.1 (E), Q3.3 (S), Q4.3 (S), U1.1 (GND), U1.22 (GND), U1.33 (GND), U2.3 (A2), U2.4 (A1), U2.5 (A0), U2.9 (VSS), U3.8 (GND)
- net PWR3/20: now also D1.2 (A)
- net Relay1: now also U2.16 (GP6), U3.1 (I1)
- net Relay2: now also U2.15 (GP5), U3.2 (I2)
- net Relay3: now also U2.14 (GP4), U3.3 (I3)
- net Relay4: now also U2.13 (GP3), U3.4 (I4)
- net Relay5: now also U2.12 (GP2), U3.5 (I5)
- net Relay6: now also U2.11 (GP1), U3.6 (I6)
- net Relay7: now also U2.10 (GP0), U3.7 (I7)
- net Temp1: now also U1.8 (IO_18/D5)
- net Temp2: now also U1.10 (IO_19/D6)
- net Temp3: now also U1.28 (IO_32)
- net VDD: now also D1.1 (K)
- net Water1: now also U1.7 (IO_35)
- net Water2: now also U1.4 (IO_36/SVP/A0)
- net Water3: now also U1.5 (IO_39/SVN)
- net at K7.2: now also U3.10 (O7)
- net at K6.2: now also U3.11 (O6)
- net at K5.2: now also U3.12 (O5)
- net at K4.2: now also U3.13 (O4)
- net at K3.2: now also U3.14 (O3)
- net at K2.2: now also U3.15 (O2)
- net at K1.2: now also U3.16 (O1)
- net at K5.1: now also J24.2 (Pin_2)
- net at K5.3: now also J24.1 (Pin_1)
- net at K5.4: now also J24.3 (Pin_3)
- net ESP_IO0 renamed DHT2
- net DHT2: now also J11.2 (Pin_2)
- new net: Q2.2 (B), R11.2
- new net: R5.2, U2.6 (~{RESET})
- new net: Q2.3 (C), Q4.1 (G), R13.1
- new net: J23.1 (Pin_1), Q4.2 (D), R13.2
- new net: J22.2 (Pin_2), Q3.2 (D), R12.2
- new net: Q1.2 (B), R10.2
- new net: Q1.3 (C), Q3.1 (G), R12.1
- new net DHT1: J19.2 (Pin_2), R9.2
- new net DISPRX: J5.7, J5.8, U1.31 (IO_16/D4)
- new net DISPTX: J5.5, J5.6, U1.29 (IO_17/D3)
- new net LED1: R10.1, U1.9 (IO_33)
- new net LED2: R11.1, U1.11 (IO_34)
- new net SCL: U1.25 (IO_22/D1/SCL), U2.1 (SCL)
- new net SDA: U1.27 (IO_21/D2/SDA), U2.2 (SDA)
- no-connect marks 16 -> 4
Other:
- note added: "DHT Sensors"
- note added: "Display Connector"
- note added: "LED"
- note added: "Power"
- note added: "Tank Level 1"
- note added: "Tank Level 2"
- note added: "Tank Level 3"
- note removed: "Temperature 4"
- note removed: "Water Level 1"
- note removed: "Water Level 2"
- note removed: "Water Level 3"
- moved on the sheet: C1, C2, J7, PS1
