File: AIO1-THT/Hardware/SmartRV-AIO-THT.kicad_sch (KiCad schematic)
At the start: 53 parts, among them J10 Temp 3, J11 Screw_Terminal_01x03, J12 Water Level Sensor, J13 Water Level Sensor, J14 Water Level Sensor, J15 Screw_Terminal_01x02, J16 Screw_Terminal_01x02, J17 Screw_Terminal_01x02, J18 Screw_Terminal_01x02, J19 Screw_Terminal_01x03, J2 Button1, J20 Screw_Terminal_01x03, J21 Screw_Terminal_01x03, J22 Screw_Terminal_01x02, J23 Screw_Terminal_01x02, J24 Screw_Terminal_01x03, J3 Button2, J4 Button3, J5 RJ45, J6 Button4, J7 Screw_Terminal_01x02, J8 Temp 1, J9 Temp 2, K1 Relay, K2 Relay, K3 Relay, K4 Relay, K5 Relay, K6 Relay, K7 Relay, Q1 2N3904, Q2 2N3904, Q3 IRF540N, Q4 IRF540N, U1 mini_esp32, U2 MCP23008-xP, U3 ULN2003

Commit message: Update
Parts:
- removed J22: Screw_Terminal_01x02, TerminalBlock_Phoenix:TerminalBlock_Phoenix_MKDS-1,5-2_1x02_P5.00mm_Horizontal, symbol Connector:Screw_Terminal_01x02
- removed Q1, Q2: 2N3904, Package_TO_SOT_THT:TO-92_Inline, symbol Transistor_BJT:2N3904
- removed Q3, Q4: IRF540N, Package_TO_SOT_THT:TO-220-3_Vertical, symbol Transistor_FET:IRF540N
- removed R10: 470, Resistor_THT:R_Axial_DIN0207_L6.3mm_D2.5mm_P7.62mm_Horizontal, symbol Device:R
- removed R12, R13: 10k, Resistor_THT:R_Axial_DIN0207_L6.3mm_D2.5mm_P7.62mm_Horizontal, symbol Device:R
- added J?: Screw_Terminal_01x02, TerminalBlock_Phoenix:TerminalBlock_Phoenix_MKDS-1,5-2_1x02_P5.00mm_Horizontal, symbol Connector:Screw_Terminal_01x02
- added Q? (x2): FQP30N06L, Package_TO_SOT_THT:TO-220-3_Vertical, symbol Transistor_FET:IRF540N
- added R?: 470, Resistor_THT:R_Axial_DIN0207_L6.3mm_D2.5mm_P7.62mm_Horizontal, symbol Device:R
Connections:
- net 12v: now also J?.2 (Pin_2)
- net GND: now also Q?.3 (S), Q?.3 (S)
- net LED1: now also R11.1
- net LED2: now also R?.1; no longer R11.1
- net at R11.2: now also Q?.1 (G)
- net at J23.1 (Pin_1): now also Q?.2 (D)
- new net: J?.1 (Pin_1), Q?.2 (D)
- new net: Q?.1 (G), R?.2
Other:
- moved on the sheet: J23, R11
